File: painel_completo/pcb4.kicad_sch (KiCad schematic)
At the start: 30 parts, among them J10 Conn_02x05_Odd_Even, J16 Conn_02x05_Odd_Even, J17 Conn_02x05_Odd_Even, J18 Conn_02x05_Odd_Even, SW1 SW_SPDT, SW10 SW_SPDT, SW11 SW_SPDT, SW12 SW_SPDT, SW2 SW_SPDT, SW3 SW_SPDT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

Commit message: adição furos fixação e alteração máscara de componentes
Parts:
- added H21, H22: MountingHole, MountingHole:MountingHole_3.2mm_M3, symbol Mechanical:MountingHole
Changed lines of the file:
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@@
     (pin "3")
+  )
+  (symbol (lib_id "Mechanical:MountingHole") (at 95.25 135.89 0) (unit 1)
+    (in_bom yes) (on_board yes) (fields_autoplaced)
+    (property "Reference" "H22" (id 0) (at 97.79 135.0553 0)
+      (effects (font (size 1.27 1.27)) (justify left))
+    )
+    (property "Value" "MountingHole" (id 1) (at 97.79 137.5922 0)
+      (effects (font (size 1.27 1.27)) (justify left))
+    )
+    (property "Footprint" "MountingHole:MountingHole_3.2mm_M3" (id 2) (at 95.25 135.89 0)
+      (effects (font (size 1.27 1.27)) hide)
+    )
+    (property "Datasheet" "~" (id 3) (at 95.25 135.89 0)
+      (effects (font (size 1.27 1.27)) hide)
+    )
   )
   (symbol (lib_id "Switch:SW_SPDT") (at 93.98 59.69 0) (unit 1)
@@
     (pin "3")
   )
+  (symbol (lib_id "Mechanical:MountingHole") (at 95.25 129.54 0) (unit 1)
+    (in_bom yes) (on_board yes) (fields_autoplaced)
+    (property "Reference" "H21" (id 0) (at 97.79 128.7053 0)
+      (effects (font (size 1.27 1.27)) (justify left))
+    )
+    (property "Value" "MountingHole" (id 1) (at 97.79 131.2422 0)
+      (effects (font (size 1.27 1.27)) (justify left))
+    )
+    (property "Footprint" "MountingHole:MountingHole_3.2mm_M3" (id 2) (at 95.25 129.54 0)
+      (effects (font (size 1.27 1.27)) hide)
+    )
+    (property "Datasheet" "~" (id 3) (at 95.25 129.54 0)
+      (effects (font (size 1.27 1.27)) hide)
+    )
+  )
   (symbol (lib_id "Device:D_Small") (at 209.55 59.69 180) (unit 1)
