File: painel_completo/painel_completo.kicad_pcb (KiCad board)
At the start: 2 copper layers, 306.3 x 296.4 mm, 171 parts, among them J1 Conn_02x05_Odd_Even, J10 Conn_02x05_Odd_Even, J11 Conn_02x10_Odd_Even, J12 Conn_02x05_Odd_Even, J13 Conn_02x02_Odd_Even, J14 Conn_02x02_Odd_Even, J15 Conn_02x10_Odd_Even, J16 Conn_02x05_Odd_Even, J17 Conn_02x05_Odd_Even, J18 Conn_02x05_Odd_Even, J19 Conn_02x10_Odd_Even, J2 Conn_02x05_Odd_Even, J3 Conn_02x06_Odd_Even, J4 Conn_02x10_Odd_Even, J5 Conn_02x03_Counter_Clockwise, J6 Conn_02x08_Counter_Clockwise, J7 Conn_02x18_Counter_Clockwise, J8 Conn_02x06_Odd_Even, J9 Conn_02x05_Odd_Even, SW1 SW_SPDT, SW10 SW_SPDT, SW11 SW_SPDT, SW12 SW_SPDT, SW13 SW_Push_LED, SW14 SW_Push_LED, SW15 SW_Push_LED, SW16 SW_Push_LED, SW17 SW_Push_LED, SW18 SW_Push_LED, SW19 SW_Push_LED, SW2 SW_SPDT, SW20 SW_Push_LED, SW21 SW_Push, SW22 SW_Push_LED, SW23 SW_Rotary3x4, SW24 SW_Rotary3x4, SW3 SW_SPDT, SW4 SW_SPDT, SW5 SW_SPDT, SW6 SW_SPDT, SW7 SW_SPDT, SW8 SW_SPDT, SW9 SW_SPDT, U1 MAX7219, U2 MAX7219, U3 74LS595, U4 74LS595, U5 Pico

Commit message: adição furos fixação e alteração máscara de componentes
Parts:
- added H19: MountingHole, MountingHole:MountingHole_3.2mm_M3, F.Cu at (205.8, 251.7)
- added H20: MountingHole, MountingHole:MountingHole_3.2mm_M3, F.Cu at (148.0, 251.7)
- added H21: MountingHole, MountingHole:MountingHole_3.2mm_M3, F.Cu at (414.8, 290.8)
- added H22: MountingHole, MountingHole:MountingHole_3.2mm_M3, F.Cu at (149.2, 288.7)
- added H23: MountingHole, MountingHole:MountingHole_3.2mm_M3, F.Cu at (284.2, 336.8)
- added H24: MountingHole, MountingHole:MountingHole_3.2mm_M3, F.Cu at (130.0, 336.2)
- added H25: MountingHole, MountingHole:MountingHole_3.2mm_M3, F.Cu at (359.2, 349.8)
- added H26: MountingHole, MountingHole:MountingHole_3.2mm_M3, F.Cu at (409.7, 352.8)
- added H27: MountingHole, MountingHole:MountingHole_3.2mm_M3, F.Cu at (399.9, 215.0)
- added H28: MountingHole, MountingHole:MountingHole_3.2mm_M3, F.Cu at (363.0, 215.0)
- added H29: MountingHole, MountingHole:MountingHole_3.2mm_M3, F.Cu at (293.8, 224.5)
- moved G*** 101.2 mm to (362.4, 73.4)
- moved H15 19.8 mm to (379.9, 316.0), turned to 180 degrees
- moved H9 17.3 mm to (148.0, 224.5), turned to 180 degrees
- moved D95 16.1 mm to (398.3, 222.5)
- moved D94 16.0 mm to (364.5, 222.5)
- moved H10 7.65 mm to (293.8, 240.8)
- moved H11 6.63 mm to (162.8, 269.0), turned to 180 degrees
- moved H18 6.58 mm to (362.8, 237.5)
- moved H17 6.53 mm to (399.9, 237.5)
- moved H12 6.40 mm to (398.7, 269.0), turned to 180 degrees
- moved H13 5.72 mm to (152.5, 316.0), turned to 180 degrees
- moved H14 5.71 mm to (269.9, 316.0), turned to 180 degrees
- moved H16 4.07 mm to (428.6, 335.4)
Routing:
- net GPIO9: track 421.9 -> 435.8 mm
- net Net-(D94-Pad1): track 30.1 -> 20.9 mm
- net Net-(D95-Pad1): track 21.6 -> 15.1 mm
- net GPIO8: track 240.3 -> 246.8 mm
- net SEG_1_B: track 238.4 -> 231.9 mm
- net DIG_2_0: track 286.8 -> 283.9 mm
- net GPIO15: track 413.6 -> 416.0 mm
- net GPIO6: track 267.6 -> 269.1 mm
- net VBUS: track 236.3 -> 237.7 mm
- net SEG_2_C: track 256.2 -> 255.0 mm
- net GPIO11: track 433.8 -> 432.7 mm
- net GPIO7: track 292.7 -> 293.5 mm
- net SEG_1_D: track 294.9 -> 295.7 mm
- net SEG_1_C: track 329.1 -> 328.4 mm
- net DIG_2_2: track 269.3 -> 269.9 mm
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Other:
- board text added: "André Biagioni andre@fiozera.com.br"
- board text added: "Felipe {dblquote}Juca{dblquote} Sanches juca@members.fsf.org"
- board text added: "Licensed under CERN-OHL-S v2 https://cern.ch/cern-ohl"
- board text added: "Setembro/2022"
- board text added: "https://forum.fiozera.com.br/t/resgate-historico-do-computador-patinho-feio-usp-1971"
- board text removed: "Setembro/2022 Felipe {dblquote}Juca{dblquote} Sanches juca@members.fsf.org https://forum.fiozera.com.br/t/resgate-historico-do-computador-patinho-feio-usp-1971"

Commit message: alteração máscara de componentes da pcb1
Other:
- board text added: "LEDs das PCBs 3, 5 e 6"
- board text added: "Licensed under CERN-OHL-S v2 or later https://cern.ch/cern-ohl"
- board text removed: "LEDs"
- board text removed: "Licensed under CERN-OHL-S v2 https://cern.ch/cern-ohl"
Changed lines of the file:
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@@
     (effects (font (size 1 1) (thickness 0.2)) (justify mirror))
   )
-  (gr_text "LEDs" (at 326.5239 129.2197 90) (layer "B.SilkS")
+  (gr_text "LEDs das PCBs 3, 5 e 6" (at 325.7296 139.446 90) (layer "B.SilkS")
     (effects (font (size 1.5 1.5) (thickness 0.3)) (justify mirror))
   )
@@
     (effects (font (size 1 1) (thickness 0.15)) (justify mirror))
   )
-  (gr_text "Licensed under CERN-OHL-S v2\nhttps://cern.ch/cern-ohl" (at 391.16 169.926) (layer "B.SilkS")
+  (gr_text "Licensed under CERN-OHL-S v2 or later\nhttps://cern.ch/cern-ohl" (at 391.16 169.926) (layer "B.SilkS")
     (effects (font (size 1 1) (thickness 0.15)) (justify left mirror))
   )
